Commit message: Add rviz2 and fix differential controller

File: urdf/rosbot3.xacro (robot description, xacro)
@@ -2,18 +2,28 @@
 <!--
   Model primitives.
-  Author: Helio Perroni Filho
+  Author: Breno Uliana de Angelo
 -->
 <robot name="rosbot3" xmlns:xacro="http://www.ros.org/wiki/xacro">
   <xacro:include filename="$(find rosbot3_description)/urdf/rosbot3.xacro"/>
   <xacro:include filename="$(find ros_commons)/urdf/gazebo.xacro"/>
-  <xacro:differential_controller
-    name="wheels_center"
-    left_joint="joint_wheel_center_left"
-    right_joint="joint_wheel_center_right"
-    wheel_separation="${wheel_separation}"
-    wheel_diameter="${wheel_diameter}"
-  />
+  <xacro:macro
+    name="add_controller"
+    params="
+      position
+      publish_odom:=false
+    "
+  >
+    <xacro:differential_controller
+      name="wheels_${position}"
+      left_joint="joint_wheel_${position}_left"
+      right_joint="joint_wheel_${position}_right"
+      wheel_separation="${chassis_width}"
+      wheel_diameter="${wheel_diameter}"
+      publish_odom="${publish_odom}"
+    />
+  </xacro:macro>
+  <xacro:add_controller position="front"/>
+  <xacro:add_controller position="rear" publish_odom="true"/>
   <xacro:remove_friction position="front"/>
-  <xacro:remove_friction position="rear"/>
   <xacro:depth_camera name="camera_front"/>
   <xacro:lidar_2d name="laser"/>

Commit message: Migrate to skid_steer_controller

File: urdf/rosbot3.xacro (robot description, xacro)
@@ -7,23 +7,14 @@
   <xacro:include filename="$(find rosbot3_description)/urdf/rosbot3.xacro"/>
   <xacro:include filename="$(find ros_commons)/urdf/gazebo.xacro"/>
-  <xacro:macro
-    name="add_controller"
-    params="
-      position
-      publish_odom:=false
-    "
-  >
-    <xacro:differential_controller
-      name="wheels_${position}"
-      left_joint="joint_wheel_${position}_left"
-      right_joint="joint_wheel_${position}_right"
-      wheel_separation="${chassis_width}"
-      wheel_diameter="${wheel_diameter}"
-      publish_odom="${publish_odom}"
-    />
-  </xacro:macro>
-  <xacro:add_controller position="front"/>
-  <xacro:add_controller position="rear" publish_odom="true"/>
-  <xacro:remove_friction position="front"/>
+  <xacro:skid_steer_controller
+    name="wheels"
+    left_joint_front="joint_wheel_front_left"
+    right_joint_front="joint_wheel_front_right"
+    left_joint_rear="joint_wheel_rear_left"
+    right_joint_rear="joint_wheel_rear_right"
+    wheel_diameter="${wheel_diameter}"
+    wheel_separation="${chassis_width}"
+    publish_odom="true"
+  />
   <xacro:depth_camera name="camera_front"/>
   <xacro:lidar_2d name="laser"/>
